File: pcb/hackpad.kicad_pcb (KiCad board)
At the start: 2 copper layers, 75 x 100 mm, 28 parts, among them J1 128x32, SW1 RotaryEncoder, U1 XIAO-RP2040-DIP

Commit message: optimize routing
Routing:
- net Encoder 0: track 21.9 -> 20.8 mm
- net Encoder 1: track 30.0 -> 29.0 mm
Changed lines of the file:
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@@
 			(remove_unused_layers no)
 		)
-		(model "${KISYS3DMOD}/Rotary_Encoder.3dshapes/RotaryEncoder_Alps_EC11E_Vertical_H20mm_CircularMountingHoles.wrl"
+		(model "C:/Users/pbhak/Downloads/EC11.STEP"
 			(offset
-				(xyz 0 0 0)
+				(xyz 7 -2.5 0)
 			)
 			(scale
@@
 			)
 			(rotate
-				(xyz 0 0 0)
+				(xyz -90 0 -90)
 			)
 		)
@@
 	)
 	(segment
-		(start 140.3 55.88)
-		(end 140.31 55.87)
-		(width 0.2)
-		(layer "F.Cu")
-		(net 1)
-	)
-	(segment
 		(start 140.31 63.49)
 		(end 178.33 63.49)
@@
 	)
 	(segment
-		(start 178.33 63.49)
-		(end 178.5 63.32)
-		(width 0.2)
-		(layer "F.Cu")
-		(net 2)
-	)
-	(segment
 		(start 141.96 50)
 		(end 142.8 50.84)
@@
 	)
 	(segment
-		(start 159.32 55.88)
-		(end 159.4 55.8)
-		(width 0.2)
-		(layer "F.Cu")
-		(net 3)
-	)
-	(segment
-		(start 178.32 55.88)
-		(end 178.5 55.7)
-		(width 0.2)
-		(layer "F.Cu")
-		(net 4)
-	)
-	(segment
 		(start 171.45 55.88)
 		(end 178.32 55.88)
@@
 	)
 	(segment
-		(start 140.27 74.93)
-		(end 140.3 74.9)
-		(width 0.2)
-		(layer "F.Cu")
-		(net 5)
-	)
-	(segment
 		(start 133.35 74.93)
 		(end 140.27 74.93)
@@
 	)
 	(segment
-		(start 159.28 74.93)
-		(end 159.32 74.89)
-		(width 0.2)
-		(layer "F.Cu")
-		(net 7)
-	)
-	(segment
 		(start 171.45 74.93)
 		(end 178.37 74.93)
@@
 	)
 	(segment
-		(start 178.37 74.93)
-		(end 178.4 74.9)
-		(width 0.2)
-		(layer "F.Cu")
-		(net 8)
-	)
-	(segment
 		(start 140.3 101.6)
 		(end 178.38 101.6)
@@
 	)
 	(segment
-		(start 178.38 101.6)
-		(end 178.4 101.62)
-		(width 0.2)
-		(layer "F.Cu")
-		(net 9)
-	)
-	(segment
 		(start 143.1791 98.7209)
 		(end 140.3 101.6)
@@
 	)
 	(segment
-		(start 140.29 93.97)
-		(end 140.3 93.98)
-		(width 0.2)
-		(layer "F.Cu")
-		(net 10)
-	)
-	(segment
 		(start 152.4 93.98)
 		(end 159.35 93.98)
@@
 	)
 	(segment
-		(start 159.35 93.98)
-		(end 159.36 93.99)
-		(width 0.2)
-		(layer "F.Cu")
-		(net 11)
-	)
-	(segment
-		(start 178.38 93.98)
-		(end 178.4 94)
-		(width 0.2)
-		(layer "F.Cu")
-		(net 12)
-	)
-	(segment
 		(start 171.45 93.98)
 		(end 178.38 93.98)
@@
 	)
 	(segment
-		(start 140.27 113.03)
-		(end 140.3 113)
-		(width 0.2)
-		(layer "F.Cu")
-		(net 13)
-	)
-	(segment
 		(start 133.35 113.03)
 		(end 140.27 113.03)
@@
 	)
 	(segment
-		(start 178.3 120.62)
-		(end 178.4 120.52)
-		(width 0.2)
-		(layer "F.Cu")
-		(net 14)
-	)
-	(segment
 		(start 144 44.42)
 		(end 141.96 42.38)
@@
 	)
 	(segment
-		(start 159.34 113.03)
-		(end 159.4 112.97)
-		(width 0.2)
-		(layer "F.Cu")
-		(net 15)
-	)
-	(segment
 		(start 171.44 113.03)
 		(end 178.27 113.03)
@@
 	)
 	(segment
-		(start 178.27 113.03)
-		(end 178.4 112.9)
-		(width 0.2)
-		(layer "F.Cu")
-		(net 16)
-	)
-	(segment
 		(start 127 58.42)
 		(end 127 115.57)
@@
 	(segment
 		(start 160.2 40.35)
-		(end 160.15 40.35)
-		(width 0.2)
-		(layer "B.Cu")
-		(net 19)
-	)
-	(segment
-		(start 160.2 40.35)
 		(end 160.2 39.4)
 		(width 0.2)
@@
 	)
 	(segment
-		(start 165.1 115.56)
-		(end 165.09 115.57)
-		(width 0.2)
-		(layer "B.Cu")
-		(net 19)
-	)
-	(segment
 		(start 139.207786 36.9)
-		(end 139.4 36.707786)
+		(end 140.007786 36.1)
 		(width 0.2)
 		(layer "B.Cu")
@@
 	)
 	(segment
-		(start 141.7 35.02)
-		(end 141.96 34.76)
-		(width 0.2)
-		(layer "B.Cu")
-		(net 21)
-	)
-	(segment
 		(start 120.8 40.3)
 		(end 124.2 36.9)
@@
 	)
 	(segment
-		(start 139.4 36.707786)
-		(end 140.007786 36.1)
-		(width 0.2)
-		(layer "B.Cu")
-		(net 21)
-	)
-	(segment
 		(start 122.9 46.56)
 		(end 124.05 47.71)
@@
 	)
 	(segment
+		(start 166.912994 50)
+		(end 168.712994 48.2)
+		(width 0.2)
+		(layer "B.Cu")
+		(net 25)
+	)
+	(segment
 		(start 178.5 48.3)
-		(end 175.4 51.4)
+		(end 178.562 48.238)
 		(width 0.2)
 		(layer "B.Cu")
@@
 	)
 	(segment
-		(start 158.6 51.4)
-		(end 157.2 50)
+		(start 178.562 43.362)
+		(end 177.2 42)
 		(width 0.2)
 		(layer "B.Cu")
@@
 	)
 	(segment
-		(start 177.2 42)
-		(end 178.5 43.3)
+		(start 178.562 48.238)
+		(end 178.562 43.362)
 		(width 0.2)
 		(layer "B.Cu")
@@
 	)
 	(segment
-		(start 178.5 43.3)
+		(start 168.712994 48.2)
+		(end 175.327 48.2)
+		(width 0.2)
+		(layer "B.Cu")
+		(net 25)
+	)
+	(segment
+		(start 157.2 50)
+		(end 166.912994 50)
+		(width 0.2)
+		(layer "B.Cu")
+		(net 25)
+	)
+	(segment
+		(start 175.427 48.3)
 		(end 178.5 48.3)
 		(width 0.2)
@@
 	)
 	(segment
-		(start 175.4 51.4)
-		(end 158.6 51.4)
+		(start 175.327 48.2)
+		(end 175.427 48.3)
 		(width 0.2)
 		(layer "B.Cu")
@@
 		(width 0.2)
 		(layer "B.Cu")
-		(net 26)
-	)
-	(segment
-		(start 158.27763 42.38)
-		(end 157.2 42.38)
-		(width 0.2)
-		(layer "B.Cu")
